File: kicad/supply.kicad_sch (KiCad schematic)
At the start: 26 parts, among them P1 USB_C_Plug_USB2.0, Q3 Si2319CDS, U10 Switch, U11 Battery, U12 AP2112K-3.3, U5 TP4056-42-ESOP8, U6 USBLC6-2P6, U7 U8205A, U8 DW01A, U9 LTC4412

Commit message: init
Parts:
- U10: symbol PCM_yvolodym:Switch small -> PCM_yvolodym:Switch_Small
Changed lines of the file:
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@@
 	)
 	(symbol
-		(lib_id "PCM_yvolodym:Switch small")
+		(lib_id "PCM_yvolodym:Switch_Small")
 		(at 160.02 138.43 0)
 		(unit 1)

Commit message: init
Parts:
- D3, D5: footprint LED_THT:LED_D2.0mm_W4.8mm_H2.5mm_FlatTop -> Diode_SMD:D_0805_2012Metric
- U10: renamed from U11; footprint PCM_yvolodym:NCR18650B -> PCM_yvolodym:CR2032
- renumbered C7 to C10, C8 to C11, C9 to C12, C4 to C7, C5 to C8, C6 to C9, U12 to U11, U5 to U4, U6 to U5, U7 to U6, U8 to U7, U9 to U8, U10 to U9
Changed lines of the file:
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@@
 			)
 		)
-		(property "Footprint" "LED_THT:LED_D2.0mm_W4.8mm_H2.5mm_FlatTop"
+		(property "Footprint" "Diode_SMD:D_0805_2012Metric"
 			(at 58.42 114.3 0)
 			(effects
@@
 		(on_board yes)
 		(dnp no)
-		(property "Reference" "U11"
+		(property "Reference" "U10"
 			(at 170.942 126.746 90)
 			(effects
@@
 			)
 		)
-		(property "Footprint" "PCM_yvolodym:NCR18650B"
+		(property "Footprint" "PCM_yvolodym:CR2032"
 			(at 165.1 130.81 0)
 			(effects
@@
 			(project "esp32-gps"
 				(path "/56168bfe-34bc-4344-8600-222c44ddf088/0856e660-1508-40ef-8651-c4510fa8d31c"
-					(reference "U11")
+					(reference "U10")
 					(unit 1)
 				)
@@
 		(dnp no)
 		(fields_autoplaced yes)
-		(property "Reference" "#PWR032"
+		(property "Reference" "#PWR030"
 			(at 196.85 95.25 0)
 			(effects
@@
 			(project "esp32-gps"
 				(path "/56168bfe-34bc-4344-8600-222c44ddf088/0856e660-1508-40ef-8651-c4510fa8d31c"
-					(reference "#PWR032")
+					(reference "#PWR030")
 					(unit 1)
 				)
@@
 		(on_board yes)
 		(dnp no)
-		(property "Reference" "C7"
+		(property "Reference" "C10"
 			(at 157.226 130.048 0)
 			(effects
@@
 			(project "esp32-gps"
 				(path "/56168bfe-34bc-4344-8600-222c44ddf088/0856e660-1508-40ef-8651-c4510fa8d31c"
-					(reference "C7")
+					(reference "C10")
 					(unit 1)
 				)
@@
 		(on_board yes)
 		(dnp no)
-		(property "Reference" "#PWR027"
+		(property "Reference" "#PWR026"
 			(at 95.25 50.8 0)
 			(effects
@@
 			(project "esp32-gps"
 				(path "/56168bfe-34bc-4344-8600-222c44ddf088/0856e660-1508-40ef-8651-c4510fa8d31c"
-					(reference "#PWR027")
+					(reference "#PWR026")
 					(unit 1)
 				)
@@
 		(dnp no)
 		(fields_autoplaced yes)
-		(property "Reference" "#PWR030"
+		(property "Reference" "#PWR028"
 			(at 104.14 29.21 0)
 			(effects
@@
 			(project "esp32-gps"
 				(path "/56168bfe-34bc-4344-8600-222c44ddf088/0856e660-1508-40ef-8651-c4510fa8d31c"
-					(reference "#PWR030")
+					(reference "#PWR028")
 					(unit 1)
 				)
@@
 		(on_board yes)
 		(dnp no)
-		(property "Reference" "U10"
+		(property "Reference" "U9"
 			(at 163.83 144.272 0)
 			(effects
@@
 			(project "esp32-gps"
 				(path "/56168bfe-34bc-4344-8600-222c44ddf088/0856e660-1508-40ef-8651-c4510fa8d31c"
-					(reference "U10")
+					(reference "U9")
 					(unit 1)
 				)
@@
 		(dnp no)
 		(fields_autoplaced yes)
-		(property "Reference" "#PWR028"
+		(property "Reference" "#PWR027"
 			(at 96.52 157.48 0)
 			(effects
@@
 			(project "esp32-gps"
 				(path "/56168bfe-34bc-4344-8600-222c44ddf088/0856e660-1508-40ef-8651-c4510fa8d31c"
-					(reference "#PWR028")
+					(reference "#PWR027")
 					(unit 1)
 				)
@@
 		(on_board yes)
 		(dnp no)
-		(property "Reference" "#PWR024"
+		(property "Reference" "#PWR023"
 			(at 58.42 87.63 0)
 			(effects
@@
 			(project "esp32-gps"
 				(path "/56168bfe-34bc-4344-8600-222c44ddf088/0856e660-1508-40ef-8651-c4510fa8d31c"
-					(reference "#PWR024")
+					(reference "#PWR023")
 					(unit 1)
 				)
@@
 		(dnp no)
 		(fields_autoplaced yes)
-		(property "Reference" "U12"
+		(property "Reference" "U11"
 			(at 173.99 24.13 0)
 			(effects
@@
 			(project "esp32-gps"
 				(path "/56168bfe-34bc-4344-8600-222c44ddf088/0856e660-1508-40ef-8651-c4510fa8d31c"
-					(reference "U12")
+					(reference "U11")
 					(unit 1)
 				)
@@
 		(on_board yes)
 		(dnp no)
-		(property "Reference" "C6"
+		(property "Reference" "C9"
 			(at 119.888 40.64 0)
 			(effects
@@
 			(project "esp32-gps"
 				(path "/56168bfe-34bc-4344-8600-222c44ddf088/0856e660-1508-40ef-8651-c4510fa8d31c"
-					(reference "C6")
+					(reference "C9")
 					(unit 1)
 				)
@@
 			)
 		)
-		(property "Footprint" "LED_THT:LED_D2.0mm_W4.8mm_H2.5mm_FlatTop"
+		(property "Footprint" "Diode_SMD:D_0805_2012Metric"
 			(at 186.69 55.88 0)
 			(effects
@@
 		(dnp no)
 		(fields_autoplaced yes)
-		(property "Reference" "#PWR031"
+		(property "Reference" "#PWR029"
 			(at 196.85 31.75 0)
 			(effects
@@
 			(project "esp32-gps"
 				(path "/56168bfe-34bc-4344-8600-222c44ddf088/0856e660-1508-40ef-8651-c4510fa8d31c"
-					(reference "#PWR031")
+					(reference "#PWR029")
 					(unit 1)
 				)
@@
 		(dnp no)
 		(fields_autoplaced yes)
-		(property "Reference" "C9"
+		(property "Reference" "C12"
 			(at 224.79 41.9099 0)
 			(effects
@@
 			(project "esp32-gps"
 				(path "/56168bfe-34bc-4344-8600-222c44ddf088/0856e660-1508-40ef-8651-c4510fa8d31c"
-					(reference "C9")
+					(reference "C12")
 					(unit 1)
 				)
@@
 		(dnp no)
 		(fields_autoplaced yes)
-		(property "Reference" "#PWR026"
+		(property "Reference" "#PWR025"
 			(at 95.25 27.94 0)
 			(effects
@@
 			(project "esp32-gps"
 				(path "/56168bfe-34bc-4344-8600-222c44ddf088/0856e660-1508-40ef-8651-c4510fa8d31c"
-					(reference "#PWR026")
+					(reference "#PWR025")
 					(unit 1)
 				)
@@
 		(dnp no)
 		(fields_autoplaced yes)
-		(property "Reference" "C8"
+		(property "Reference" "C11"
 			(at 200.66 44.4499 0)
 			(effects
@@
 			(project "esp32-gps"
 				(path "/56168bfe-34bc-4344-8600-222c44ddf088/0856e660-1508-40ef-8651-c4510fa8d31c"
-					(reference "C8")
+					(reference "C11")
 					(unit 1)
 				)
@@
 		(on_board yes)
 		(dnp no)
-		(property "Reference" "U8"
+		(property "Reference" "U7"
 			(at 132.08 113.03 0)
 			(effects
@@
 			(project "esp32-gps"
 				(path "/56168bfe-34bc-4344-8600-222c44ddf088/0856e660-1508-40ef-8651-c4510fa8d31c"
-					(reference "U8")
+					(reference "U7")
 					(unit 1)
 				)
@@
 		(on_board yes)
 		(dnp no)
-		(property "Reference" "U7"
+		(property "Reference" "U6"
 			(at 123.19 141.732 90)
 			(effects
@@
 			(project "esp32-gps"
 				(path "/56168bfe-34bc-4344-8600-222c44ddf088/0856e660-1508-40ef-8651-c4510fa8d31c"
-					(reference "U7")
+					(reference "U6")
 					(unit 1)
 				)
@@
 		(dnp no)
 		(fields_autoplaced yes)
-		(property "Reference" "#PWR023"
+		(property "Reference" "#PWR022"
 			(at 54.61 81.28 0)
 			(effects
@@
 			(project "esp32-gps"
 				(path "/56168bfe-34bc-4344-8600-222c44ddf088/0856e660-1508-40ef-8651-c4510fa8d31c"
-					(reference "#PWR023")
+					(reference "#PWR022")
 					(unit 1)
 				)
@@
 		(on_board yes)
 		(dnp no)
-		(property "Reference" "U9"
+		(property "Reference" "U8"
 			(at 131.572 71.374 0)
 			(effects
@@
 			(project "esp32-gps"
 				(path "/56168bfe-34bc-4344-8600-222c44ddf088/0856e660-1508-40ef-8651-c4510fa8d31c"
-					(reference "U9")
+					(reference "U8")
 					(unit 1)
 				)
@@
 		(dnp no)
 		(fields_autoplaced yes)
-		(property "Reference" "U5"
+		(property "Reference" "U4"
 			(at 83.4233 119.38 0)
 			(effects
@@
 			(project "esp32-gps"
 				(path "/56168bfe-34bc-4344-8600-222c44ddf088/0856e660-1508-40ef-8651-c4510fa8d31c"
-					(reference "U5")
+					(reference "U4")
 					(unit 1)
 				)
@@
 		(dnp no)
 		(fields_autoplaced yes)
-		(property "Reference" "#PWR034"
+		(property "Reference" "#PWR032"
 			(at 220.98 55.88 0)
 			(effects
@@
 			(project "esp32-gps"
 				(path "/56168bfe-34bc-4344-8600-222c44ddf088/0856e660-1508-40ef-8651-c4510fa8d31c"
-					(reference "#PWR034")
+					(reference "#PWR032")
 					(unit 1)
 				)
@@
 		(dnp no)
 		(fields_autoplaced yes)
-		(property "Reference" "#PWR025"
+		(property "Reference" "#PWR024"
 			(at 81.28 106.68 0)
 			(effects
@@
 			(project "esp32-gps"
 				(path "/56168bfe-34bc-4344-8600-222c44ddf088/0856e660-1508-40ef-8651-c4510fa8d31c"
-					(reference "#PWR025")
+					(reference "#PWR024")
 					(unit 1)
 				)
@@
 		(on_board yes)
 		(dnp no)
-		(property "Reference" "C4"
+		(property "Reference" "C7"
 			(at 64.008 101.092 0)
 			(effects
@@
 			(project "esp32-gps"
 				(path "/56168bfe-34bc-4344-8600-222c44ddf088/0856e660-1508-40ef-8651-c4510fa8d31c"
-					(reference "C4")
+					(reference "C7")
 					(unit 1)
 				)
@@
 		(on_board yes)
 		(dnp no)
-		(property "Reference" "U6"
+		(property "Reference" "U5"
 			(at 101.346 40.386 0)
 			(effects
@@
 			(project "esp32-gps"
 				(path "/56168bfe-34bc-4344-8600-222c44ddf088/0856e660-1508-40ef-8651-c4510fa8d31c"
-					(reference "U6")
+					(reference "U5")
 					(unit 1)
 				)
@@
 		(dnp no)
 		(fields_autoplaced yes)
-		(property "Reference" "#PWR033"
+		(property "Reference" "#PWR031"
 			(at 220.98 41.91 0)
 			(effects
@@
 			(project "esp32-gps"
 				(path "/56168bfe-34bc-4344-8600-222c44ddf088/0856e660-1508-40ef-8651-c4510fa8d31c"
-					(reference "#PWR033")
+					(reference "#PWR031")
 					(unit 1)
 				)
@@
 		(on_board yes)
 		(dnp no)
-		(property "Reference" "C5"
+		(property "Reference" "C8"
 			(at 109.728 138.938 0)
 			(effects
@@
 			(project "esp32-gps"
 				(path "/56168bfe-34bc-4344-8600-222c44ddf088/0856e660-1508-40ef-8651-c4510fa8d31c"
-					(reference "C5")
+					(reference "C8")
 					(unit 1)
 				)

Commit message: init
Parts:
- renumbered C9 to C10, C10 to C11, C11 to C12, C12 to C13, C7 to C8, C8 to C9, R12 to R15, R13 to R16, R14 to R17, R15 to R18, R16 to R19, R17 to R20, R18 to R21
Changed lines of the file:
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@@
 		(dnp no)
 		(fields_autoplaced yes)
-		(property "Reference" "#PWR030"
+		(property "Reference" "#PWR034"
 			(at 196.85 95.25 0)
 			(effects
@@
 			(project "esp32-gps"
 				(path "/56168bfe-34bc-4344-8600-222c44ddf088/0856e660-1508-40ef-8651-c4510fa8d31c"
-					(reference "#PWR030")
+					(reference "#PWR034")
 					(unit 1)
 				)
@@
 		(on_board yes)
 		(dnp no)
-		(property "Reference" "C10"
+		(property "Reference" "C11"
 			(at 157.226 130.048 0)
 			(effects
@@
 			(project "esp32-gps"
 				(path "/56168bfe-34bc-4344-8600-222c44ddf088/0856e660-1508-40ef-8651-c4510fa8d31c"
-					(reference "C10")
+					(reference "C11")
 					(unit 1)
 				)
@@
 		(on_board yes)
 		(dnp no)
-		(property "Reference" "#PWR026"
+		(property "Reference" "#PWR030"
 			(at 95.25 50.8 0)
 			(effects
@@
 			(project "esp32-gps"
 				(path "/56168bfe-34bc-4344-8600-222c44ddf088/0856e660-1508-40ef-8651-c4510fa8d31c"
-					(reference "#PWR026")
+					(reference "#PWR030")
 					(unit 1)
 				)
@@
 		(dnp no)
 		(fields_autoplaced yes)
-		(property "Reference" "#PWR028"
+		(property "Reference" "#PWR032"
 			(at 104.14 29.21 0)
 			(effects
@@
 			(project "esp32-gps"
 				(path "/56168bfe-34bc-4344-8600-222c44ddf088/0856e660-1508-40ef-8651-c4510fa8d31c"
-					(reference "#PWR028")
+					(reference "#PWR032")
 					(unit 1)
 				)
@@
 		(dnp no)
 		(fields_autoplaced yes)
-		(property "Reference" "#PWR027"
+		(property "Reference" "#PWR031"
 			(at 96.52 157.48 0)
 			(effects
@@
 			(project "esp32-gps"
 				(path "/56168bfe-34bc-4344-8600-222c44ddf088/0856e660-1508-40ef-8651-c4510fa8d31c"
-					(reference "#PWR027")
+					(reference "#PWR031")
 					(unit 1)
 				)
@@
 		(on_board yes)
 		(dnp no)
-		(property "Reference" "#PWR023"
+		(property "Reference" "#PWR027"
 			(at 58.42 87.63 0)
 			(effects
@@
 			(project "esp32-gps"
 				(path "/56168bfe-34bc-4344-8600-222c44ddf088/0856e660-1508-40ef-8651-c4510fa8d31c"
-					(reference "#PWR023")
+					(reference "#PWR027")
 					(unit 1)
 				)
@@
 		(dnp no)
 		(fields_autoplaced yes)
-		(property "Reference" "R15"
+		(property "Reference" "R18"
 			(at 99.06 142.2399 0)
 			(effects
@@
 			(project "esp32-gps"
 				(path "/56168bfe-34bc-4344-8600-222c44ddf088/0856e660-1508-40ef-8651-c4510fa8d31c"
-					(reference "R15")
+					(reference "R18")
 					(unit 1)
 				)
@@
 		(on_board yes)
 		(dnp no)
-		(property "Reference" "C9"
+		(property "Reference" "C10"
 			(at 119.888 40.64 0)
 			(effects
@@
 			(project "esp32-gps"
 				(path "/56168bfe-34bc-4344-8600-222c44ddf088/0856e660-1508-40ef-8651-c4510fa8d31c"
-					(reference "C9")
+					(reference "C10")
 					(unit 1)
 				)
@@
 		(dnp no)
 		(fields_autoplaced yes)
-		(property "Reference" "#PWR029"
+		(property "Reference" "#PWR033"
 			(at 196.85 31.75 0)
 			(effects
@@
 			(project "esp32-gps"
 				(path "/56168bfe-34bc-4344-8600-222c44ddf088/0856e660-1508-40ef-8651-c4510fa8d31c"
-					(reference "#PWR029")
+					(reference "#PWR033")
 					(unit 1)
 				)
@@
 		(dnp no)
 		(fields_autoplaced yes)
-		(property "Reference" "R17"
+		(property "Reference" "R20"
 			(at 158.75 114.3 90)
 			(effects
@@
 			(project "esp32-gps"
 				(path "/56168bfe-34bc-4344-8600-222c44ddf088/0856e660-1508-40ef-8651-c4510fa8d31c"
-					(reference "R17")
+					(reference "R20")
 					(unit 1)
 				)
@@
 		(dnp no)
 		(fields_autoplaced yes)
-		(property "Reference" "C12"
+		(property "Reference" "C13"
 			(at 224.79 41.9099 0)
 			(effects
@@
 			(project "esp32-gps"
 				(path "/56168bfe-34bc-4344-8600-222c44ddf088/0856e660-1508-40ef-8651-c4510fa8d31c"
-					(reference "C12")
+					(reference "C13")
 					(unit 1)
 				)
@@
 		(dnp no)
 		(fields_autoplaced yes)
-		(property "Reference" "R16"
+		(property "Reference" "R19"
 			(at 120.65 133.3499 0)
 			(effects
@@
 			(project "esp32-gps"
 				(path "/56168bfe-34bc-4344-8600-222c44ddf088/0856e660-1508-40ef-8651-c4510fa8d31c"
-					(reference "R16")
+					(reference "R19")
 					(unit 1)
 				)
@@
 		(dnp no)
 		(fields_autoplaced yes)
-		(property "Reference" "#PWR025"
+		(property "Reference" "#PWR029"
 			(at 95.25 27.94 0)
 			(effects
@@
 			(project "esp32-gps"
 				(path "/56168bfe-34bc-4344-8600-222c44ddf088/0856e660-1508-40ef-8651-c4510fa8d31c"
-					(reference "#PWR025")
+					(reference "#PWR029")
 					(unit 1)
 				)
@@
 		(dnp no)
 		(fields_autoplaced yes)
-		(property "Reference" "C11"
+		(property "Reference" "C12"
 			(at 200.66 44.4499 0)
 			(effects
@@
 			(project "esp32-gps"
 				(path "/56168bfe-34bc-4344-8600-222c44ddf088/0856e660-1508-40ef-8651-c4510fa8d31c"
-					(reference "C11")
+					(reference "C12")
 					(unit 1)
 				)
@@
 		(on_board yes)
 		(dnp no)
-		(property "Reference" "R13"
+		(property "Reference" "R16"
 			(at 73.152 33.02 90)
 			(effects
@@
 			(project "esp32-gps"
 				(path "/56168bfe-34bc-4344-8600-222c44ddf088/0856e660-1508-40ef-8651-c4510fa8d31c"
-					(reference "R13")
+					(reference "R16")
 					(unit 1)
 				)
@@
 		(on_board yes)
 		(dnp no)
-		(property "Reference" "R14"
+		(property "Reference" "R17"
 			(at 73.152 40.64 90)
 			(effects
@@
 			(project "esp32-gps"
 				(path "/56168bfe-34bc-4344-8600-222c44ddf088/0856e660-1508-40ef-8651-c4510fa8d31c"
-					(reference "R14")
+					(reference "R17")
 					(unit 1)
 				)
@@
 		(dnp no)
 		(fields_autoplaced yes)
-		(property "Reference" "#PWR022"
+		(property "Reference" "#PWR026"
 			(at 54.61 81.28 0)
 			(effects
@@
 			(project "esp32-gps"
 				(path "/56168bfe-34bc-4344-8600-222c44ddf088/0856e660-1508-40ef-8651-c4510fa8d31c"
-					(reference "#PWR022")
+					(reference "#PWR026")
 					(unit 1)
 				)
@@
 		(dnp no)
 		(fields_autoplaced yes)
-		(property "Reference" "#PWR032"
+		(property "Reference" "#PWR036"
 			(at 220.98 55.88 0)
 			(effects
@@
 			(project "esp32-gps"
 				(path "/56168bfe-34bc-4344-8600-222c44ddf088/0856e660-1508-40ef-8651-c4510fa8d31c"
-					(reference "#PWR032")
+					(reference "#PWR036")
 					(unit 1)
 				)
@@
 		(dnp no)
 		(fields_autoplaced yes)
-		(property "Reference" "#PWR024"
+		(property "Reference" "#PWR028"
 			(at 81.28 106.68 0)
 			(effects
@@
 			(project "esp32-gps"
 				(path "/56168bfe-34bc-4344-8600-222c44ddf088/0856e660-1508-40ef-8651-c4510fa8d31c"
-					(reference "#PWR024")
+					(reference "#PWR028")
 					(unit 1)
 				)
@@
 		(on_board yes)
 		(dnp no)
-		(property "Reference" "R18"
+		(property "Reference" "R21"
 			(at 180.848 43.18 0)
 			(effects
@@
 			(project "esp32-gps"
 				(path "/56168bfe-34bc-4344-8600-222c44ddf088/0856e660-1508-40ef-8651-c4510fa8d31c"
-					(reference "R18")
+					(reference "R21")
 					(unit 1)
 				)
@@
 		(on_board yes)
 		(dnp no)
-		(property "Reference" "C7"
+		(property "Reference" "C8"
 			(at 64.008 101.092 0)
 			(effects
@@
 			(project "esp32-gps"
 				(path "/56168bfe-34bc-4344-8600-222c44ddf088/0856e660-1508-40ef-8651-c4510fa8d31c"
-					(reference "C7")
+					(reference "C8")
 					(unit 1)
 				)
@@
 		(dnp no)
 		(fields_autoplaced yes)
-		(property "Reference" "R12"
+		(property "Reference" "R15"
 			(at 60.96 125.7299 0)
 			(effects
@@
 			(project "esp32-gps"
 				(path "/56168bfe-34bc-4344-8600-222c44ddf088/0856e660-1508-40ef-8651-c4510fa8d31c"
-					(reference "R12")
+					(reference "R15")
 					(unit 1)
 				)
@@
 		(dnp no)
 		(fields_autoplaced yes)
-		(property "Reference" "#PWR031"
+		(property "Reference" "#PWR035"
 			(at 220.98 41.91 0)
 			(effects
@@
 			(project "esp32-gps"
 				(path "/56168bfe-34bc-4344-8600-222c44ddf088/0856e660-1508-40ef-8651-c4510fa8d31c"
-					(reference "#PWR031")
+					(reference "#PWR035")
 					(unit 1)
 				)
@@
 		(on_board yes)
 		(dnp no)
-		(property "Reference" "C8"
+		(property "Reference" "C9"
 			(at 109.728 138.938 0)
 			(effects
@@
 			(project "esp32-gps"
 				(path "/56168bfe-34bc-4344-8600-222c44ddf088/0856e660-1508-40ef-8651-c4510fa8d31c"
-					(reference "C8")
+					(reference "C9")
 					(unit 1)
 				)
