File: kicad/esp32-gps.kicad_sch (KiCad schematic)
At the start: 30 parts, among them J1 Conn_01x07_Socket, Q1 BCW66G, Q2 BCW66G, SW1 RESET, SW2 BOOT, U1 ESP32-PICO-V3, U2 CH340C

Commit message: init
Parts:
- removed J1: Conn_01x07_Socket, Connector_PinSocket_2.54mm:PinSocket_1x07_P2.54mm_Vertical, symbol Connector:Conn_01x07_Socket
- removed TP1: TestPoint, TestPoint:TestPoint_Pad_3.0x3.0mm, symbol Connector:TestPoint
- added J1, J2: Conn_Coaxial_Small, Connector_Coaxial:U.FL_Molex_MCRF_73412-0110_Vertical, symbol Connector:Conn_Coaxial_Small
- added U3: GP-01, PCM_yvolodym:GP-01, symbol PCM_yvolodym:GP-01
Connections:
- net +3.3V: now also U3.23 (3V3)
- net GND: now also J1.2 (Ext), J2.2 (Ext), U3.10 (GND), U3.12 (GND), U3.13 (GND)
- net at C2.1, C3.1: now also J1.1 (In)
- new net: J2.1 (In), U3.11 (RF)
Other:
- note removed: "CS"
- note removed: "DC"
- note removed: "GND"
- note removed: "RST"
- note removed: "SCL"
- note removed: "SOA [MOSI]"
- note removed: "VCC"

Commit message: init
Connections:
- net GND: now also U3.24 (GND)
- net GPS_TX: now reaches U3.20 (TX0)
- net GPS_TX: now also U1.14 (IO25)
- net GPS_RX: now reaches U3.21 (RX0)
- net GPS_RX: now also U1.15 (IO26)
- no-connect marks 24 -> 22
Changed lines of the file:
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@@
-	)
-	(no_connect
-		(at 106.68 118.11)
 	)
 	(no_connect
@@
 	)
 	(no_connect
-		(at 106.68 120.65)
-	)
-	(no_connect
 		(at 106.68 90.17)
 	)
@@
 		(pts
 			(xy 86.36 64.77) (xy 86.36 62.23)
+		)
+		(stroke
+			(width 0)
+			(type default)
+		)
+	)
+	(wire
+		(pts
+			(xy 106.68 118.11) (xy 111.76 118.11)
+		)
+		(stroke
+			(width 0)
+			(type default)
+		)
+	)
+	(wire
+		(pts
+			(xy 106.68 120.65) (xy 111.76 120.65)
+		)
+		(stroke
+			(width 0)
+			(type default)
+		)
+	)
+	(wire
+		(pts
+			(xy 165.1 139.7) (xy 170.18 139.7)
+		)
+		(stroke
+			(width 0)
+			(type default)
+		)
+	)
+	(wire
+		(pts
+			(xy 165.1 142.24) (xy 170.18 142.24)
+		)
+		(stroke
+			(width 0)
+			(type default)
+		)
+	)
+	(wire
+		(pts
+			(xy 165.1 149.86) (xy 170.18 149.86)
+		)
+		(stroke
+			(width 0)
+			(type default)
+		)
+	)
+	(wire
+		(pts
+			(xy 170.18 149.86) (xy 170.18 152.4)
 		)
 		(stroke
@@
 	(label "RTS"
 		(at 116.84 97.79 0)
+		(effects
+			(font
+				(size 1.27 1.27)
+			)
+			(justify left bottom)
+		)
+	)
+	(label "GPS_TX"
+		(at 111.76 118.11 0)
+		(effects
+			(font
+				(size 1.27 1.27)
+			)
+			(justify left bottom)
+		)
+	)
+	(label "GPS_RX"
+		(at 111.76 120.65 0)
+		(effects
+			(font
+				(size 1.27 1.27)
+			)
+			(justify left bottom)
+		)
+	)
+	(label "GPS_TX"
+		(at 170.18 139.7 0)
+		(effects
+			(font
+				(size 1.27 1.27)
+			)
+			(justify left bottom)
+		)
+	)
+	(label "GPS_RX"
+		(at 170.18 142.24 0)
 		(effects
 			(font
@@
 					(unit 1)
 				)
+			)
+		)
+	)
+	(symbol
+		(lib_id "power:GND")
+		(at 170.18 152.4 0)
+		(unit 1)
+		(exclude_from_sim no)
+		(in_bom yes)
+		(on_board yes)
+		(dnp no)
+		(fields_autoplaced yes)
+		(property "Reference" "#PWR018"
+			(at 170.18 158.75 0)
+			(effects
+				(font
+					(size 1.27 1.27)
+				)
+				(hide yes)
+			)
+		)
+		(property "Value" "GND"
+			(at 170.18 157.48 0)
+			(effects
+				(font
+					(size 1.27 1.27)
+				)
+			)
+		)
+		(property "Footprint" ""
+			(at 170.18 152.4 0)
+			(effects
+				(font
+					(size 1.27 1.27)
+				)
+				(hide yes)
+			)
+		)
+		(property "Datasheet" ""
+			(at 170.18 152.4 0)
+			(effects
+				(font
+					(size 1.27 1.27)
+				)
+				(hide yes)
+			)
+		)
+		(property "Description" "Power symbol creates a global label with name \"GND\" , ground"
+			(at 170.18 152.4 0)
+			(effects
+				(font
+					(size 1.27 1.27)
+				)
+				(hide yes)
+			)
+		)
+		(pin "1"
+		)
+		(instances
+			(project "esp32-gps"
+				(path "/56168bfe-34bc-4344-8600-222c44ddf088"
+					(reference "#PWR018")
+					(unit 1)
+				)

Commit message: init
Connections:
- net +3.3V: now also U3.22 (VRTC)
- no-connect marks 22 -> 29
Changed lines of the file:
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@@
+	)
+	(no_connect
+		(at 142.24 127)
+	)
+	(no_connect
+		(at 142.24 132.08)
+	)
+	(no_connect
+		(at 142.24 139.7)
+	)
+	(no_connect
+		(at 142.24 142.24)
+	)
+	(no_connect
+		(at 165.1 124.46)
+	)
+	(no_connect
+		(at 165.1 129.54)
+	)
+	(no_connect
+		(at 165.1 132.08)
 	)
 	(no_connect
@@
 	)
 	(wire
+		(pts
+			(xy 165.1 144.78) (xy 165.1 147.32)
+		)
+		(stroke
+			(width 0)
+			(type default)
+		)
+	)
+	(junction
+		(at 165.1 147.32)
+		(diameter 0)
+		(color 0 0 0 0)
+	)
+	(wire

Commit message: init
Connections:
- net DTR: no longer Q2.3 (E)
- net GND: now also Q1.3 (E), Q2.3 (E)
- net RTS: no longer Q1.3 (E)
- no-connect marks 29 -> 34
Changed lines of the file:
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@@
 	(paper "A4")
 	(junction
-		(at 223.52 133.35)
-		(diameter 0)
-		(color 0 0 0 0)
-	)
-	(junction
 		(at 43.18 69.85)
 		(diameter 0)
@@
 	)
 	(junction
-		(at 219.71 114.3)
-		(diameter 0)
-		(color 0 0 0 0)
-	)
-	(junction
 		(at 53.34 172.72)
 		(diameter 0)
@@
 	)
 	(no_connect
+		(at 106.68 87.63)
+	)
+	(no_connect
+		(at 106.68 105.41)
+	)
+	(no_connect
+		(at 106.68 115.57)
+	)
+	(no_connect
+		(at 106.68 113.03)
+	)
+	(no_connect
+		(at 106.68 110.49)
+	)
+	(no_connect
 		(at 251.46 50.8)
 	)
@@
 	(wire
 		(pts
-			(xy 245.11 124.46) (xy 219.71 124.46)
+			(xy 245.11 124.46) (xy 252.73 124.46)
 		)
 		(stroke
@@
 	(wire
 		(pts
-			(xy 219.71 124.46) (xy 219.71 114.3)
-		)
-		(stroke
-			(width 0)
-			(type default)
-		)
-	)
-	(wire
-		(pts
 			(xy 106.68 97.79) (xy 116.84 97.79)
 		)
@@
 	(wire
 		(pts
+			(xy 252.73 121.92) (xy 252.73 124.46)
+		)
+		(stroke
+			(width 0)
+			(type default)
+		)
+	)
+	(junction
+		(at 252.73 124.46)
+		(diameter 0)
+		(color 0 0 0 0)
+	)
+	(wire
+		(pts
 			(xy 165.1 144.78) (xy 165.1 147.32)
 		)
@@
 	(wire
 		(pts
-			(xy 245.11 121.92) (xy 223.52 121.92)
+			(xy 245.11 121.92) (xy 252.73 121.92)
 		)
 		(stroke
@@
 	(wire
 		(pts
-			(xy 223.52 121.92) (xy 223.52 133.35)
-		)
-		(stroke
-			(width 0)
-			(type default)
-		)
-	)
-	(wire
-		(pts
 			(xy 223.52 48.26) (xy 231.14 48.26)
 		)
@@
 					(unit 1)
 				)
+			)
+		)
+	)
+	(symbol
+		(lib_id "power:GND")
+		(at 252.73 124.46 0)
+		(unit 1)
+		(exclude_from_sim no)
+		(in_bom yes)
+		(on_board yes)
+		(dnp no)
+		(fields_autoplaced yes)
+		(property "Reference" "#PWR019"
+			(at 252.73 130.81 0)
+			(effects
+				(font
+					(size 1.27 1.27)
+				)
+				(hide yes)
+			)
+		)
+		(property "Value" "GND"
+			(at 252.73 129.54 0)
+			(effects
+				(font
+					(size 1.27 1.27)
+				)
+			)
+		)
+		(property "Footprint" ""
+			(at 252.73 124.46 0)
+			(effects
+				(font
+					(size 1.27 1.27)
+				)
+				(hide yes)
+			)
+		)
+		(property "Datasheet" ""
+			(at 252.73 124.46 0)
+			(effects
+				(font
+					(size 1.27 1.27)
+				)
+				(hide yes)
+			)
+		)
+		(property "Description" "Power symbol creates a global label with name \"GND\" , ground"
+			(at 252.73 124.46 0)
+			(effects
+				(font
+					(size 1.27 1.27)
+				)
+				(hide yes)
+			)
+		)
+		(pin "1"
+		)
+		(instances
+			(project "esp32-gps"
+				(path "/56168bfe-34bc-4344-8600-222c44ddf088"
+					(reference "#PWR019")
+					(unit 1)
+				)

Commit message: init
Parts:
- renumbered C11 to C2, C2 to C3, C3 to C4, C1 to C5, C12 to C6, R8 to R10, R9 to R11, R1 to R2, R2 to R3, R2 to R4, R3 to R5, R4 to R6, R5 to R7, R6 to R8, R7 to R9, U3 to U2, U2 to U3

Commit message: init
Parts:
- removed U3: CH340C, Package_SO:SOIC-16_3.9x9.9mm_P1.27mm, symbol Interface_USB:CH340C
- added U3: CP2102N-Axx-xQFN28, Package_DFN_QFN:QFN-28-1EP_5x5mm_P0.5mm_EP3.35x3.35mm, symbol Interface_USB:CP2102N-Axx-xQFN28
- renumbered C6 to C5, C5 to C6
Connections:
- net +3.3V: now also U3.6 (VDD), U3.7 (VREGIN)
- net CTS: now also U3.23 (~{CTS})
- net DTR: now also U3.28 (~{DTR})
- net GND: now also U3.29 (GND), U3.3 (GND)
- net RTS: now also U3.24 (~{RTS})
- net Supply/D+: now also U3.4 (D+)
- net Supply/D-: now also U3.5 (D-)
- net at R10.1: now also U3.26 (TXD)
- net at R11.1: now also U3.25 (RXD)
- no-connect marks 34 -> 31
Other:
- moved on the sheet: C5, Q1, Q2, R8, R9

Commit message: init
Parts:
- added C6: 4,7µF, Capacitor_SMD:C_0805_2012Metric, symbol Device:C
- added R10: 1K, Resistor_SMD:R_0805_2012Metric, symbol Device:R
- added R8: 22.1K, Resistor_SMD:R_0805_2012Metric, symbol Device:R
- added R9: 47.5K, Resistor_SMD:R_0805_2012Metric, symbol Device:R
- renumbered C6 to C7, R8 to R11, R9 to R12, R10 to R13, R11 to R14
Connections:
- net +3.3V: now also C6.1, R10.2
- net GND: now also C6.2, R9.1
- net at U3.8 (VBUS): now also R8.1, R9.2
- net at U3.9 (~{RST}): now also R10.1
- new net +5V: R8.2
- no-connect marks 31 -> 30
Other:
- moved on the sheet: C5

Commit message: init
Connections:
- no-connect marks 30 -> 45
Changed lines of the file:
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@@
+	)
+	(no_connect
+		(at 259.08 87.63)
 	)
 	(no_connect
@@
 	)
 	(no_connect
+		(at 259.08 67.31)
+	)
+	(no_connect
 		(at 165.1 132.08)
 	)
 	(no_connect
 		(at 165.1 129.54)
+	)
+	(no_connect
+		(at 259.08 64.77)
 	)
 	(no_connect
@@
 	)
 	(no_connect
+		(at 259.08 77.47)
+	)
+	(no_connect
+		(at 259.08 49.53)
+	)
+	(no_connect
 		(at 106.68 113.03)
 	)
 	(no_connect
+		(at 259.08 41.91)
+	)
+	(no_connect
 		(at 106.68 125.73)
+	)
+	(no_connect
+		(at 259.08 74.93)
 	)
 	(no_connect
@@
 	)
 	(no_connect
+		(at 259.08 54.61)
+	)
+	(no_connect
 		(at 106.68 80.01)
 	)
 	(no_connect
 		(at 106.68 128.27)
+	)
+	(no_connect
+		(at 259.08 72.39)
+	)
+	(no_connect
+		(at 259.08 57.15)
 	)
 	(no_connect
@@
 	)
 	(no_connect
+		(at 259.08 62.23)
+	)
+	(no_connect
 		(at 142.24 139.7)
 	)
 	(no_connect
 		(at 106.68 105.41)
+	)
+	(no_connect
+		(at 259.08 46.99)
+	)
+	(no_connect
+		(at 259.08 82.55)
 	)
 	(no_connect
@@
 	)
 	(no_connect
+		(at 259.08 69.85)
+	)
+	(no_connect
 		(at 106.68 90.17)
 	)
@@
 	)
 	(no_connect
+		(at 259.08 85.09)
+	)
+	(no_connect
