File: kicad/esp32-gps.kicad_pcb (KiCad board)
At the start: 2 copper layers, 56.5 x 50 mm, 57 parts, among them J1 Conn_Coaxial_Small, J2 Conn_Coaxial_Small, P1 USB_C_Plug_USB2.0, Q1 BCW66G, Q2 BCW66G, Q3 Si2319CDS, SW1 RESET, SW2 BOOT, U1 ESP32-PICO-V3, U10 Battery, U11 AP2112K-3.3, U2 GP-01, U3 CH340C, U4 TP4056-42-ESOP8, U5 USBLC6-2P6, U6 U8205A, U7 DW01A, U8 LTC4412, U9 Switch

Commit message: init
Parts:
- U3: value CH340C -> CP2102N-Axx-xQFN28; footprint Package_SO:SOIC-16_3.9x9.9mm_P1.27mm -> Package_DFN_QFN:QFN-28-1EP_5x5mm_P0.5mm_EP3.35x3.35mm
- moved R11 37.1 mm to (184.3, 78.8)
- moved R10 37.1 mm to (184.3, 75.9)
- moved U3 1.23 mm to (178.5, 78.0), turned to 0 degrees
- renumbered C6 to C5, C5 to C6
Connections:
- U3 pad 1: GND -> unconnected-(U3-~{DCD}-Pad1)
- U3 pad 13: /DTR -> unconnected-(U3-CHREN-Pad13)
- U3 pad 14: /RTS -> unconnected-(U3-CHR1-Pad14)
- U3 pad 16: +3.3V -> unconnected-(U3-~{WAKEUP}/GPIO.3-Pad16)
- U3 pad 2: Net-(U3-TXD) -> unconnected-(U3-~{RI}/CLK-Pad2)
- U3 pad 3: Net-(U3-RXD) -> GND
- U3 pad 4: +3.3V -> /Supply/D+
- U3 pad 5: /Supply/D+ -> /Supply/D-
- U3 pad 6: /Supply/D- -> +3.3V
- U3 pad 7: unconnected-(U3-NC-Pad7) -> +3.3V
- U3 pad 9: /CTS -> unconnected-(U3-~{RST}-Pad9)

Commit message: init
Parts:
- added C6: 4,7µF, Capacitor_SMD:C_0805_2012Metric, F.Cu at (176.6, 84.0)
- added R10: 1K, Resistor_SMD:R_0805_2012Metric, F.Cu at (172.1, 89.9)
- added R8: 22.1K, Resistor_SMD:R_0805_2012Metric, F.Cu at (172.1, 84.0)
- added R9: 47.5K, Resistor_SMD:R_0805_2012Metric, F.Cu at (172.1, 86.9)
- renumbered C9 to C10, C10 to C11, C11 to C12, C12 to C13, C6 to C7, C7 to C8, C8 to C9, R8 to R11, R9 to R12, R10 to R13, R11 to R14, R12 to R15, R13 to R16, R14 to R17, R15 to R18, R16 to R19, R17 to R20, R18 to R21
Connections:
- U3 pad 8: unconnected-(U3-VBUS-Pad8) -> Net-(U3-VBUS)
- U3 pad 9: unconnected-(U3-~{RST}-Pad9) -> Net-(U3-~{RST})

Commit message: init
Parts:
- moved J2 48.7 mm to (151.0, 74.5)
- moved J1 47.4 mm to (134.5, 110.5)
- moved U5 44.0 mm to (178.6, 95.0)
- moved C6 42.8 mm to (135.4, 96.0)
- moved R17 42.8 mm to (184.0, 95.1), turned to 90 degrees
- moved R13 37.4 mm to (179.6, 113.0)
- moved SW2 36.5 mm to (146.1, 107.7)
- moved SW1 36.3 mm to (146.1, 102.7)
- moved U1 34.5 mm to (137.2, 102.7)
- moved R20 33.7 mm to (175.0, 79.4), turned to 90 degrees
- moved R16 33.7 mm to (173.4, 94.0)
- moved U4 32.6 mm to (168.0, 77.6)
- moved D3 32.3 mm to (162.0, 77.9), turned to 90 degrees
- moved R18 31.3 mm to (174.5, 83.9), turned to 90 degrees
- moved R14 31.0 mm to (172.5, 107.5), turned to 90 degrees
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
Commit message: init
Parts:
- moved R11 34.4 mm to (155.0, 90.5)
- moved R17 25.4 mm to (159.0, 90.5)
- moved U3 24.4 mm to (156.0, 97.5)
- moved Q1 24.0 mm to (163.0, 92.5)
- moved R8 23.0 mm to (161.0, 103.5), turned to -90 degrees
- moved R13 22.0 mm to (163.5, 98.0), turned to -90 degrees
- moved R18 19.6 mm to (155.0, 85.6)
- moved R20 17.2 mm to (159.0, 85.6)
- moved R9 14.6 mm to (168.5, 102.0), turned to 180 degrees
- moved C8 13.1 mm to (158.9, 74.0)
- moved C12 11.7 mm to (175.5, 101.0)
- moved U6 11.5 mm to (174.0, 81.0)
- moved R12 10.6 mm to (176.5, 111.6), turned to 90 degrees
- moved U7 10.2 mm to (174.0, 75.0)
- moved R16 8.89 mm to (176.0, 85.5), turned to 180 degrees
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Routing:
- net +3.3V: track 0.00 -> 143.5 mm, vias 0 -> 8
- net +5V: track 0.00 -> 127.1 mm, vias 0 -> 6
- net /HVBAT: track 0.00 -> 69.3 mm, vias 0 -> 2
- net Net-(U6-S2): track 0.00 -> 67.3 mm, vias 0 -> 3
- net /RTS: track 0.00 -> 62.5 mm, vias 0 -> 4
- net /EN: track 0.00 -> 59.6 mm, vias 0 -> 2
- net /IO0: track 0.00 -> 52.5 mm, vias 0 -> 2
- net Net-(U1-LNA_IN): track 0.00 -> 47.5 mm, vias 0 -> 2
- net /TXD0: track 0.00 -> 47.1 mm, vias 0 -> 2
- net Net-(U1-SENSOR_VP): track 0.00 -> 40.7 mm, vias 0 -> 3
- net Net-(U10--): track 0.00 -> 36.2 mm, vias 0 -> 2
- net Net-(P1-CC): track 0.00 -> 36.1 mm, vias 0 -> 2
- net Net-(D4-K): track 0.00 -> 35.7 mm, vias 0 -> 2
- net GND: track 0.00 -> 32.4 mm, vias 0 -> 9
- net /GPS_TX: track 0.00 -> 31.0 mm
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- added copper zone on F.Cu, net GND
Other:
- board size 56.5 x 50 mm -> 50 x 50 mm
- copper layers 2 -> 4

Commit message: init
Routing:
- net Net-(U3-RXD): track 0.00 -> 40.5 mm, vias 0 -> 2
- net Net-(U3-TXD): track 11.5 -> 13.6 mm
- net /RTS: track 62.5 -> 64.4 mm
Changed lines of the file:
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@@
+	)
+	(segment
+		(start 158.1 93.751471)
+		(end 157.748529 93.4)
+		(width 0.2)
+		(layer "F.Cu")
+		(net 29)
+	)
+	(segment
+		(start 158.5 94)
+		(end 158.1 94)
+		(width 0.2)
+		(layer "F.Cu")
+		(net 29)
 	)
 	(segment
@@
 	)
 	(segment
+		(start 156.6 94.334315)
+		(end 156.6 94.3942)
+		(width 0.2)
+		(layer "F.Cu")
+		(net 29)
+	)
+	(segment
+		(start 156.5 94.4942)
+		(end 156.5 95.05)
+		(width 0.2)
+		(layer "F.Cu")
+		(net 29)
+	)
+	(segment
 		(start 137.91 106.11)
 		(end 137.91 106.9197)
@@
 	)
 	(segment
-		(start 156.5 95.05)
+		(start 157.251471 93.4)
+		(end 156.9 93.751471)
+		(width 0.2)
+		(layer "F.Cu")
+		(net 29)
+	)
+	(segment
+		(start 158.1 94)
+		(end 158.1 93.751471)
+		(width 0.2)
+		(layer "F.Cu")
+		(net 29)
+	)
+	(segment
+		(start 156.6 94.3942)
 		(end 156.5 94.4942)
 		(width 0.2)
@@
 	)
 	(segment
-		(start 156.5 94.4942)
-		(end 156.152 94.1462)
+		(start 157.748529 93.4)
+		(end 157.251471 93.4)
+		(width 0.2)
+		(layer "F.Cu")
+		(net 29)
+	)
+	(segment
+		(start 156.9 94.034315)
+		(end 156.6 94.334315)
 		(width 0.2)
 		(layer "F.Cu")
@@
 		(net 29)
 	)
+	(segment
+		(start 156.9 93.751471)
+		(end 156.9 94.034315)
+		(width 0.2)
+		(layer "F.Cu")
+		(net 29)
+	)
 	(via
 		(at 175.5869 113.4131)
@@
 	)
 	(via
-		(at 156.152 94.1462)
+		(at 158.5 94)
 		(size 0.6)
 		(drill 0.3)
@@
 		(drill 0.3)
 		(layers "F.Cu" "B.Cu")
-		(net 29)
-	)
-	(segment
-		(start 156.152 94.1462)
-		(end 158.2662 96.2604)
-		(width 0.2)
-		(layer "In1.Cu")
 		(net 29)
 	)
@@
 	)
 	(segment
+		(start 158.5 96.0266)
+		(end 158.2662 96.2604)
+		(width 0.2)
+		(layer "In1.Cu")
+		(net 29)
+	)
+	(segment
+		(start 158.5 94)
+		(end 158.5 96.0266)
+		(width 0.2)
+		(layer "In1.Cu")
+		(net 29)
+	)
+	(segment
 		(start 142.1296 111.202529)
 		(end 141.778129 111.554)
@@
 	)
 	(segment
-		(start 156.854 93)
-		(end 156.3555 93.4985)
+		(start 155.214386 94.35)
+		(end 155.425 94.560614)
+		(width 0.2)
+		(layer "F.Cu")
+		(net 30)
+	)
+	(segment
+		(start 157.923129 93)
+		(end 154.5 93)
+		(width 0.2)
+		(layer "F.Cu")
+		(net 30)
+	)
+	(segment
+		(start 163.4735 96.4559)
+		(end 160.0592 93.0416)
+		(width 0.2)
+		(layer "F.Cu")
+		(net 30)
+	)
+	(segment
+		(start 155.5 94.9263)
+		(end 155.5 95.05)
+		(width 0.2)
+		(layer "F.Cu")
+		(net 30)
+	)
+	(segment
+		(start 163.4735 97.0644)
+		(end 163.4735 96.4559)
+		(width 0.2)
+		(layer "F.Cu")
+		(net 30)
+	)
+	(segment
+		(start 155.425 94.560614)
+		(end 155.425 94.8513)
+		(width 0.2)
+		(layer "F.Cu")
+		(net 30)
+	)
+	(segment
+		(start 155.425 94.8513)
+		(end 155.5 94.9263)
+		(width 0.2)
+		(layer "F.Cu")
+		(net 30)
+	)
+	(segment
+		(start 154.5 93)
+		(end 154.5 93.9263)
 		(width 0.2)
 		(layer "F.Cu")
@@
 	)
 	(segment
-		(start 163.4735 97.0644)
-		(end 163.4735 96.4559)
-		(width 0.2)
-		(layer "F.Cu")
-		(net 30)
-	)
-	(segment
-		(start 163.4735 96.4559)
-		(end 160.0592 93.0416)
+		(start 154.5 93.9263)
+		(end 154.9237 94.35)
+		(width 0.2)
+		(layer "F.Cu")
+		(net 30)
+	)
+	(segment
+		(start 154.9237 94.35)
+		(end 155.214386 94.35)
 		(width 0.2)
 		(layer "F.Cu")
@@
 	)
 	(segment
-		(start 156.3555 93.4985)
-		(end 155.9278 93.4985)
-		(width 0.2)
-		(layer "F.Cu")
-		(net 30)
-	)
-	(segment
-		(start 155.5 93.9263)
-		(end 155.5 95.05)
-		(width 0.2)
-		(layer "F.Cu")
-		(net 30)
-	)
-	(segment
-		(start 157.923129 93)
-		(end 156.854 93)
-		(width 0.2)
-		(layer "F.Cu")
-		(net 30)
-	)
-	(segment
-		(start 155.9278 93.4985)
-		(end 155.5 93.9263)
-		(width 0.2)
-		(layer "F.Cu")
-		(net 30)
-	)
-	(segment
+		(start 156 94)
+		(end 156 95.05)
+		(width 0.2)
+		(layer "F.Cu")
+		(net 31)
+	)
+	(via
+		(at 172.5 112.5)
+		(size 0.6)
+		(drill 0.3)
+		(layers "F.Cu" "B.Cu")
+		(net 31)
+	)
+	(via
+		(at 156 94)
+		(size 0.6)
+		(drill 0.3)
+		(layers "F.Cu" "B.Cu")
+		(net 31)
+	)
+	(segment
+		(start 157.251471 112.647842)
+		(end 157.251471 95.251471)
+		(width 0.2)
+		(layer "In1.Cu")
+		(net 31)
+	)
+	(segment
+		(start 162.521629 117.2705)
+		(end 161.874129 117.2705)
+		(width 0.2)
+		(layer "In1.Cu")
+		(net 31)
+	)
+	(segment
+		(start 172.5 114.215229)
+		(end 170.843529 115.8717)
+		(width 0.2)
+		(layer "In1.Cu")
+		(net 31)
+	)
+	(segment
+		(start 157.251471 95.251471)
+		(end 156 94)
+		(width 0.2)
+		(layer "In1.Cu")
+		(net 31)
+	)
+	(segment
+		(start 170.843529 115.8717)
+		(end 163.920429 115.8717)
+		(width 0.2)
+		(layer "In1.Cu")
+		(net 31)
+	)
+	(segment
+		(start 161.874129 117.2705)
+		(end 157.251471 112.647842)
+		(width 0.2)
+		(layer "In1.Cu")
+		(net 31)
+	)
+	(segment
+		(start 172.5 112.5)
+		(end 172.5 114.215229)
+		(width 0.2)
+		(layer "In1.Cu")
+		(net 31)
+	)
+	(segment
+		(start 163.920429 115.8717)
+		(end 162.521629 117.2705)
+		(width 0.2)
+		(layer "In1.Cu")
+		(net 31)
+	)
+	(segment
+		(start 156.636523 93.5)
+		(end 156.736523 93.6)
+		(width 0.2)
+		(layer "In2.Cu")
+		(net 31)
+	)
+	(segment

Commit message: init
Parts:
- J1, J2: value Conn_Coaxial_Small -> MHF4; footprint Connector_Coaxial:U.FL_Molex_MCRF_73412-0110_Vertical -> PCM_yvolodym:MHF4
- moved Q2 5.09 mm to (171.0, 106.5)
- moved R21 5.02 mm to (176.5, 106.0), turned to -90 degrees
- moved J2 1.58 mm to (149.5, 75.0)
- moved J1 1.12 mm to (134.0, 111.5)
- turned C12 to 180 degrees
- turned R14 to -90 degrees
- turned R15 to 90 degrees
- turned R2 to 180 degrees
Routing:
- net +3.3V: track 143.5 -> 0.00 mm, vias 8 -> 0
- net +5V: track 127.1 -> 0.00 mm, vias 6 -> 0
- net /HVBAT: track 69.3 -> 0.00 mm, vias 2 -> 0
- net Net-(U6-S2): track 67.3 -> 0.00 mm, vias 3 -> 0
- net /RTS: track 64.4 -> 0.00 mm, vias 4 -> 0
- net /EN: track 59.6 -> 0.00 mm, vias 2 -> 0
- net /IO0: track 52.5 -> 0.00 mm, vias 2 -> 0
- net Net-(U1-LNA_IN): track 47.5 -> 0.00 mm, vias 2 -> 0
- net /TXD0: track 47.1 -> 0.00 mm, vias 2 -> 0
- net Net-(U1-SENSOR_VP): track 40.7 -> 0.00 mm, vias 3 -> 0
- net Net-(U3-RXD): track 40.5 -> 0.00 mm, vias 2 -> 0
- net Net-(U10--): track 36.2 -> 0.00 mm, vias 2 -> 0
- net Net-(P1-CC): track 36.1 -> 0.00 mm, vias 2 -> 0
- net Net-(D4-K): track 35.7 -> 0.00 mm, vias 2 -> 0
- net GND: track 32.4 -> 0.00 mm, vias 9 -> 0
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
Commit message: init
Parts:
- moved R16 14.9 mm to (158.6, 104.0)
- moved R7 5.39 mm to (171.0, 87.5)
- moved C4 4.76 mm to (169.0, 83.0)
- moved R14 3.16 mm to (164.0, 102.5)
- moved C5 2.95 mm to (132.5, 92.5)
- moved C6 2.95 mm to (132.5, 96.0)
- moved U5 2.42 mm to (134.8, 102.5), turned to 90 degrees
- moved R2 2.20 mm to (163.1, 83.0)
- moved R10 2.06 mm to (137.9, 92.5)
- moved C9 1.97 mm to (138.0, 96.0)
- moved R19 1.50 mm to (176.0, 88.5), turned to -90 degrees
- moved R12 0.59 mm to (143.9, 92.5)
- moved R13 0.50 mm to (144.0, 96.0)
- renumbered C9 to C1, C3 to C10, C10 to C11, C5 to C13, C8 to C3, C11 to C4, C13 to C5, C4 to C8, C1 to C9, D3 to D1, D5 to D3, D1 to D5, J2 to J1, J1 to J2, Q3 to Q2, Q2 to Q3, R20 to R1, R7 to R10, R17 to R11, R4 to R12, R5 to R13, R8 to R14, R13 to R15, R6 to R16, R14 to R17, R12 to R18, R10 to R19, R19 to R2, R21 to R20, R9 to R21, R18 to R3, R2 to R4, R1 to R5, R15 to R6, R16 to R7, R3 to R8, R11 to R9, U2 to U1, U9 to U10, U10 to U11, U7 to U2, U4 to U3, U6 to U4, U1 to U5, U8 to U6, U3 to U7, U11 to U8, U5 to U9

Commit message: init
Parts:
- moved C10 36.9 mm to (132.4, 100.0)
- moved R16 25.7 mm to (174.0, 113.0), turned to 0 degrees
- moved U1 21.6 mm to (156.1, 98.8)
- moved R17 20.5 mm to (157.2, 111.0), turned to -90 degrees
- moved Q3 19.8 mm to (149.5, 104.0)
- moved R14 18.4 mm to (163.5, 95.5), turned to 180 degrees
- moved R12 17.4 mm to (164.0, 99.5), turned to -90 degrees
- moved R21 15.5 mm to (161.0, 105.0), turned to 180 degrees
- moved R9 14.6 mm to (170.5, 87.5)
- moved U3 14.6 mm to (170.6, 96.0), turned to 90 degrees
- moved R13 14.5 mm to (149.0, 97.5)
- moved D2 14.2 mm to (138.0, 99.5)
- moved SW2 13.9 mm to (132.5, 105.0), turned to 90 degrees
- moved R6 13.6 mm to (154.5, 91.0)
- moved C9 11.7 mm to (153.5, 85.5), turned to -90 degrees
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- renumbered C9 to C1, C11 to C10, C4 to C11, C5 to C13, C10 to C3, C8 to C4, C13 to C5, C3 to C8, C1 to C9, D5 to D1, D1 to D3, D3 to D5, J2 to J1, J1 to J2, Q3 to Q2, Q2 to Q3, R5 to R1, R19 to R10, R9 to R11, R18 to R12, R15 to R13, R17 to R14, R6 to R15, R7 to R16, R11 to R17, R3 to R18, R2 to R19, R4 to R2, R1 to R20, R20 to R21, R8 to R3, R12 to R4, R13 to R5, R16 to R6, R10 to R7, R14 to R8, R21 to R9, U5 to U1, U11 to U10, U8 to U11, U1 to U2, U7 to U3, U3 to U4, U9 to U5, U4 to U6, U2 to U7, U6 to U8, U10 to U9
Routing:
- net +3.3V: track 0.00 -> 161.7 mm, vias 0 -> 5
- net +5V: track 0.00 -> 130.0 mm, vias 0 -> 4
- net /IO0: track 0.00 -> 64.0 mm, vias 0 -> 3
- net /EN: track 0.00 -> 63.6 mm, vias 0 -> 3
- net /HVBAT: track 0.00 -> 58.8 mm, vias 0 -> 3
- net Net-(U6-S2): track 0.00 -> 58.2 mm, vias 0 -> 2
- net GND: track 0.00 -> 58.0 mm, vias 0 -> 8
- net /TXD0: track 0.00 -> 45.5 mm, vias 0 -> 4
- net Net-(J1-SIGNAL): track 0.00 -> 39.9 mm, vias 0 -> 3
- net Net-(U10--): track 0.00 -> 35.6 mm, vias 0 -> 2
- net Net-(U1-SENSOR_VP): track 0.00 -> 35.5 mm, vias 0 -> 2
- net /GPS_TX: track 0.00 -> 34.1 mm, vias 0 -> 2
- net Net-(U3-VBUS): track 0.00 -> 32.1 mm
- net Net-(U1-LNA_IN): track 0.00 -> 31.3 mm, vias 0 -> 2
- net /GPS_RX: track 0.00 -> 28.8 mm, vias 0 -> 2
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