File: kicad/esp32-gps.kicad_pcb (KiCad board)
At the start: 4 copper layers, 50 x 50 mm, 61 parts, among them J1 MHF4, J2 MHF4, P1 USB_C_Plug_USB2.0, Q1 BCW66G, Q2 BCW66G, Q3 Si2319CDS, SW1 RESET, SW2 BOOT, U1 ESP32-PICO-V3, U10 Battery, U11 AP2112K-3.3, U2 GP-01, U3 CP2102N-Axx-xQFN28, U4 TP4056-42-ESOP8, U5 USBLC6-2P6, U6 U8205A, U7 DW01A, U8 LTC4412, U9 Switch

Commit message: init
Routing:
- net GND: track 58.0 -> 153.0 mm, vias 8 -> 23
- net Net-(U10--): track 35.6 -> 29.3 mm
- net +3.3V: track 161.7 -> 165.9 mm

Commit message: init
Routing:
- net GND: track 153.0 -> 155.7 mm
Changed lines of the file:
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@@
+	)
+	(segment
+		(start 160.755 113.32)
+		(end 160.18 113.895)
+		(width 0.2)
+		(layer "F.Cu")
+		(net 1)
 	)
 	(segment
@@
 	)
 	(segment
+		(start 167.7 113.32)
+		(end 168.245 113.32)
+		(width 0.2)
+		(layer "F.Cu")
+		(net 1)
+	)
+	(segment
 		(start 154.5 82.9)
 		(end 154.95 83.35)
@@
 		(width 0.2)
 		(layer "F.Cu")
+		(net 1)
+	)
+	(segment
+		(start 161.3 113.32)
+		(end 160.755 113.32)
+		(width 0.2)
+		(layer "F.Cu")
+		(net 1)
+	)
+	(segment
+		(start 168.245 113.32)
+		(end 168.82 113.895)
+		(width 0.2)
+		(layer "F.Cu")

Commit message: init
Parts:
- renumbered C9 to C1, C4 to C10, C7 to C11, C5 to C13, C8 to C3, C11 to C4, C1 to C5, C10 to C6, C13 to C7, C6 to C8, C3 to C9, D3 to D1, D1 to D3, D5 to D4, D4 to D5, J2 to J1, J1 to J2, Q3 to Q1, Q1 to Q2, Q2 to Q3, R3 to R1, R7 to R11, R4 to R12, R21 to R14, R14 to R15, R6 to R16, R5 to R17, R17 to R18, R12 to R19, R18 to R2, R8 to R20, R16 to R21, R1 to R3, R20 to R4, R2 to R5, R15 to R6, R19 to R7, R11 to R8, SW2 to SW1, SW1 to SW2, U2 to U1, U9 to U10, U10 to U11, U7 to U2, U4 to U3, U6 to U4, U1 to U5, U8 to U6, U3 to U7, U11 to U8, U5 to U9

Commit message: init
Routing:
- net Net-(U10--): track 29.3 -> 0.00 mm, vias 2 -> 0
- net GND: track 155.7 -> 154.7 mm
Changed lines of the file:
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@@
 	)
 	(segment
-		(start 154.2 82.35)
-		(end 153.75 82.35)
+		(start 152.5125 82.35)
+		(end 154.2 82.35)
 		(width 0.2)
 		(layer "F.Cu")
@@
 	)
 	(segment
-		(start 142.95 88.55)
-		(end 142.95 89.55)
-		(width 0.2)
-		(layer "F.Cu")
-		(net 1)
-	)
-	(segment
 		(start 154.5 82.35)
 		(end 154.35 82.5)
@@
 	)
 	(segment
-		(start 153.75 82.35)
-		(end 152.5125 82.35)
-		(width 0.2)
-		(layer "F.Cu")
-		(net 1)
-	)
-	(segment
 		(start 138.95 96)
 		(end 138 95.05)
@@
 	)
 	(segment
-		(start 154.25 115.4667)
-		(end 154.25 116.74)
-		(width 0.2)
-		(layer "F.Cu")
-		(net 91)
-	)
-	(via
-		(at 154.25 115.4667)
-		(size 0.6)
-		(drill 0.3)
-		(layers "F.Cu" "B.Cu")
-		(net 91)
-	)
-	(via
-		(at 154.2505 87.4857)
-		(size 0.6)
-		(drill 0.3)
-		(layers "F.Cu" "B.Cu")
-		(net 91)
-	)
-	(segment
-		(start 154.2505 87.4857)
-		(end 154.2505 115.4662)
-		(width 0.2)
-		(layer "In1.Cu")
-		(net 91)
-	)
-	(segment
-		(start 154.2505 115.4662)
-		(end 154.25 115.4667)
-		(width 0.2)
-		(layer "In1.Cu")
-		(net 91)
-	)
-	(segment
